File: Eagle files/BarGraphDriver.sch (EAGLE design)
At the start: 22 parts, among them IC1 74HC595D, IC2 74HC595D

Commit message: aaaaaaaaaaaaaaaaaaaaaaaaaaaaaaaaaaaa
Cleaned up schematics, replaced wire solder points with header pin
mounts for standardization, recreated a broken file and dealt with the
confusion and insanity that followed.
Parts:
- removed GND, GND1, RCLK, RCLK1, SER, SRCLK, SRCLK1, S_OUT: WIREPAD2,15/1,0, wirepad:WIREPAD2,15/1,0
- removed VCC, VCC1: WIREPAD2,15/1,0, smallWirepadSquare:WIREPAD2,15/1,0
- added PAD1: (no value), wirepad:SMD2
- added SR_IN, SR_OUT: (no value), SparkFun-Connectors:M05PTH
Connections:
- removed net SER: IC1A.SER, SER.P
- removed net SRCLK: IC1A.SCK, IC2A.SCK, SRCLK.P, SRCLK1.P
- removed net S_OUT: IC2A.QH*, S_OUT.P
- new net SCLK: IC1A.SCK, IC2A.SCK, SR_IN.3, SR_OUT.3
- new net SER_IN: IC1A.SER, SR_IN.4
- new net SER_OUT: IC2A.QH*, SR_OUT.4
- net GND: now also PAD1.P, SR_IN.5, SR_OUT.5; no longer GND.P, GND1.P
- net RCLK: now also SR_IN.2, SR_OUT.2; no longer RCLK.P, RCLK1.P
- net VCC: now also SR_IN.1, SR_OUT.1; no longer VCC.P, VCC1.P
Other:
- moved on the sheet: IC2P
