File: Eagle files/main_board.sch (EAGLE design)
At the start: 21 parts

Commit message: aaaaaaaaaaaaaaaaaaaaaaaaaaaaaaaaaaaa
Cleaned up schematics, replaced wire solder points with header pin
mounts for standardization, recreated a broken file and dealt with the
confusion and insanity that followed.
Connections:
- net IRSIG renamed IRSENSE
- removed net N$28: T1.7
- new net N$5: T1.5
- net IRLED: now also T1.7; no longer T1.5
Changed lines of the file:
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@@
-</segment>
-</net>
-<net name="N$28" class="0">
-<segment>
-<pinref part="T1" gate="G$1" pin="7"/>
-<wire x1="-12.7" y1="58.42" x2="-20.32" y2="58.42" width="0.1524" layer="91"/>
 </segment>
 </net>
@@
 <net name="IRLED" class="0">
 <segment>
-<pinref part="T1" gate="G$1" pin="5"/>
-<wire x1="-12.7" y1="53.34" x2="-20.32" y2="53.34" width="0.1524" layer="91"/>
-<label x="-17.78" y="53.34" size="1.778" layer="95"/>
-</segment>
-<segment>
 <pinref part="USB2" gate="G$1" pin="GND_DRAIN"/>
 <wire x1="144.78" y1="63.5" x2="162.56" y2="63.5" width="0.1524" layer="91"/>
@@
 <label x="144.78" y="30.48" size="1.778" layer="95"/>
 </segment>
+<segment>
+<pinref part="T1" gate="G$1" pin="7"/>
+<wire x1="-12.7" y1="58.42" x2="-20.32" y2="58.42" width="0.1524" layer="91"/>
+<label x="-17.78" y="58.42" size="1.778" layer="95"/>
+</segment>
 </net>
 <net name="DATA_OUT_2" class="0">
@@
 </segment>
 </net>
-<net name="IRSIG" class="0">
+<net name="IRSENSE" class="0">
 <segment>
 <pinref part="SHOULDER1" gate="G$1" pin="1"/>
@@
 </segment>
 </net>
+<net name="N$5" class="0">
+<segment>
+<pinref part="T1" gate="G$1" pin="5"/>
+<wire x1="-12.7" y1="53.34" x2="-20.32" y2="53.34" width="0.1524" layer="91"/>
+</segment>
+</net>
