File: Eagle files/LaserModule.brd (EAGLE design)
At the start: 100 x 80 mm, 6 parts, among them Q1 IRF510

Commit message: New Lazer
Changed some stuff in the laser module, nbd.
Parts:
- removed GND_BATT, GND_IN, SINGAL_IN, VCC_BATT: WIREPAD2,54/1,1, wirepad:2,54/1,1
- added BATT, SIG: (no value), SparkFun-Connectors:1X02
Connections:
- removed net N$1: Q1.1, SINGAL_IN.1
- removed net N$3: TSAL6000.A, VCC_BATT.1
- new net SIG: Q1.1, SIG.2
- new net VCC: BATT.2, TSAL6000.A
- net GND: now also BATT.1, SIG.1; no longer GND_BATT.1, GND_IN.1
Routing:
- net N$3: track 38.2 -> 0.00 mm
- net VCC: track 0.00 -> 38.1 mm
- net N$1: track 27.8 -> 0.00 mm
- net SIG: track 0.00 -> 26.1 mm
- net GND: track 5.08 -> 0.00 mm, vias 22 -> 20
Other:
- board size 100 x 80 mm -> 17.8 x 41.9 mm
- board text added: "+"
- board text added: "-"
- board text added: "Greg T - v1.2"
- board text added: "Lazer Module"
- board text added: "~"
- board text removed: "+BATT"
- board text removed: "-BATT"
- board text removed: "GND"
- board text removed: "IR LED"
- board text removed: "LaserModule v1.1"
- board text removed: "S_IN"

Commit message: Fixes
more fixes >:|
should e ready for fabbing
Changed lines of the file:
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@@
 <?xml version="1.0" encoding="utf-8"?>
 <!DOCTYPE eagle SYSTEM "eagle.dtd">
-<eagle version="7.5.0">
+<eagle version="7.4.0">
 <drawing>
 <settings>
@@
 <contactref element="Q1" pad="2"/>
 <contactref element="TSAL6000" pad="K"/>
-<wire x1="57.15" y1="27.94" x2="57.15" y2="22.86" width="0.6096" layer="1"/>
-<wire x1="57.15" y1="22.86" x2="55.88" y2="21.59" width="0.6096" layer="1"/>
+<wire x1="57.15" y1="27.94" x2="57.15" y2="22.86" width="1.016" layer="1"/>
+<wire x1="57.15" y1="22.86" x2="55.88" y2="21.59" width="1.016" layer="1"/>
 </signal>
 <signal name="GND">
