File: Eagle files/main_board.brd (EAGLE design)
At the start: 88.6 x 66 mm, 21 parts

Commit message: aaaaaaaaaaaaaaaaaaaaaaaaaaaaaaaaaaaa
Cleaned up schematics, replaced wire solder points with header pin
mounts for standardization, recreated a broken file and dealt with the
confusion and insanity that followed.
Connections:
- net IRSIG renamed IRSENSE
- removed net N$28: T1.7
- new net N$5: T1.5
- net IRLED: now also T1.7; no longer T1.5
Routing:
- net IRLED: track 102.4 -> 102.5 mm, vias 3 -> 2
- net GND: vias 15 -> 17
Changed lines of the file:
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@@
 <via x="13.335" y="31.75" extent="1-16" drill="0.6" shape="square"/>
 <via x="14.605" y="13.335" extent="1-16" drill="0.6" shape="square"/>
+<via x="33.02" y="19.685" extent="1-16" drill="0.6" shape="square"/>
+<via x="26.67" y="22.225" extent="1-16" drill="0.6" shape="square"/>
+<wire x1="41.275" y1="27.94" x2="33.655" y2="27.94" width="0" layer="19" extent="1-1"/>
 </signal>
 <signal name="N$1">
@@
 <via x="13.6525" y="2.8575" extent="1-16" drill="0.6096"/>
 </signal>
-<signal name="N$28">
-<contactref element="T1" pad="7"/>
-</signal>
 <signal name="MEMCS">
 <contactref element="T1" pad="8"/>
@@
 </signal>
 <signal name="IRLED">
-<contactref element="T1" pad="5"/>
 <contactref element="USB2" pad="GND_DRAIN"/>
 <contactref element="USB1" pad="GND_DRAIN"/>
+<contactref element="T1" pad="7"/>
 <wire x1="16.1925" y1="19.685" x2="7.62" y2="11.1125" width="0.4064" layer="1"/>
-<wire x1="16.1925" y1="35.2425" x2="16.1925" y2="19.685" width="0.4064" layer="1"/>
-<wire x1="16.51" y1="35.56" x2="16.1925" y2="35.2425" width="0.4064" layer="1"/>
+<wire x1="16.1925" y1="30.1625" x2="16.1925" y2="19.685" width="0.4064" layer="1"/>
+<wire x1="19.3675" y1="33.3375" x2="16.1925" y2="30.1625" width="0.4064" layer="1"/>
+<wire x1="21.59" y1="35.56" x2="19.3675" y2="33.3375" width="0.4064" layer="16"/>
 <wire x1="7.62" y1="11.1125" x2="7.62" y2="10.92" width="0.4064" layer="1"/>
 <wire x1="59.055" y1="10.795" x2="81.28" y2="10.795" width="0.4064" layer="16"/>
@@
 <wire x1="52.07" y1="17.145" x2="52.705" y2="17.145" width="0.4064" layer="16"/>
 <wire x1="49.53" y1="19.685" x2="52.07" y2="17.145" width="0.4064" layer="16"/>
-<wire x1="43.18" y1="19.685" x2="49.53" y2="19.685" width="0.4064" layer="16"/>
-<wire x1="38.735" y1="15.24" x2="43.18" y2="19.685" width="0.4064" layer="1"/>
-<wire x1="38.735" y1="14.9225" x2="38.735" y2="15.24" width="0.4064" layer="16"/>
-<wire x1="37.465" y1="13.6525" x2="38.735" y2="14.9225" width="0.4064" layer="16"/>
-<wire x1="35.8775" y1="13.6525" x2="37.465" y2="13.6525" width="0.4064" layer="16"/>
-<wire x1="29.845" y1="19.685" x2="35.8775" y2="13.6525" width="0.4064" layer="16"/>
-<wire x1="16.1925" y1="19.685" x2="29.845" y2="19.685" width="0.4064" layer="16"/>
+<wire x1="43.4975" y1="19.685" x2="49.53" y2="19.685" width="0.4064" layer="16"/>
+<wire x1="39.37" y1="23.8125" x2="43.4975" y2="19.685" width="0.4064" layer="16"/>
+<wire x1="39.37" y1="27.305" x2="39.37" y2="23.8125" width="0.4064" layer="16"/>
+<wire x1="36.195" y1="27.305" x2="39.37" y2="27.305" width="0.4064" layer="1"/>
+<wire x1="34.29" y1="29.21" x2="36.195" y2="27.305" width="0.4064" layer="1"/>
+<wire x1="27.94" y1="29.21" x2="34.29" y2="29.21" width="0.4064" layer="1"/>
+<wire x1="21.59" y1="35.56" x2="27.94" y2="29.21" width="0.4064" layer="1"/>
 <wire x1="81.28" y1="10.795" x2="81.28" y2="10.67" width="0.4064" layer="16"/>
-<via x="43.18" y="19.685" extent="1-16" drill="0.6096"/>
-<via x="38.735" y="15.24" extent="1-16" drill="0.6096"/>
-<via x="16.1925" y="19.685" extent="1-16" drill="0.6096"/>
+<via x="19.3675" y="33.3375" extent="1-16" drill="0.6096"/>
+<via x="39.37" y="27.305" extent="1-16" drill="0.6096"/>
 </signal>
 <signal name="DATA_OUT_2">
@@
 <wire x1="46.99" y1="6.35" x2="41.91" y2="6.35" width="0.4064" layer="16"/>
 </signal>
-<signal name="IRSIG">
+<signal name="IRSENSE">
 <contactref element="SHOULDER1" pad="1"/>
 <contactref element="IRSENSE" pad="3"/>
-<contactref element="T1" pad="6"/>
 <contactref element="SHOULDER2" pad="6"/>
-<wire x1="4.7625" y1="49.8475" x2="19.05" y2="35.56" width="0.4064" layer="1"/>
 <wire x1="4.7625" y1="54.2925" x2="4.7625" y2="49.8475" width="0.4064" layer="1"/>
 <wire x1="11.43" y1="60.96" x2="4.7625" y2="54.2925" width="0.4064" layer="1"/>
@@
 <wire x1="46.355" y1="26.035" x2="51.1175" y2="21.2725" width="0.4064" layer="16"/>
 <wire x1="28.575" y1="26.035" x2="46.355" y2="26.035" width="0.4064" layer="1"/>
-<wire x1="19.05" y1="35.56" x2="28.575" y2="26.035" width="0.4064" layer="1"/>
 <wire x1="61.9125" y1="63.8175" x2="64.77" y2="60.96" width="0.4064" layer="1"/>
 <wire x1="14.2875" y1="63.8175" x2="61.9125" y2="63.8175" width="0.4064" layer="1"/>
 <wire x1="11.43" y1="60.96" x2="14.2875" y2="63.8175" width="0.4064" layer="1"/>
 <via x="46.355" y="26.035" extent="1-16" drill="0.6096"/>
+<contactref element="T1" pad="6"/>
+<wire x1="28.575" y1="26.035" x2="19.05" y2="35.56" width="0.4064" layer="1"/>
+<wire x1="4.7625" y1="49.8475" x2="19.05" y2="35.56" width="0.4064" layer="1"/>
 </signal>
 <signal name="LEDBLUE">
@@
 <via x="58.1025" y="19.685" extent="1-16" drill="0.6096"/>
 </signal>
+<signal name="N$5">
+<contactref element="T1" pad="5"/>
+</signal>
 </signals>

Commit message: Fixes
more fixes >:|
should e ready for fabbing
Changed lines of the file:
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@@
 <?xml version="1.0" encoding="utf-8"?>
 <!DOCTYPE eagle SYSTEM "eagle.dtd">
-<eagle version="7.5.0">
+<eagle version="7.4.0">
 <drawing>
 <settings>
@@
 <layer number="43" name="vRestrict" color="2" fill="10" visible="yes" active="yes"/>
 <layer number="44" name="Drills" color="7" fill="1" visible="no" active="yes"/>
-<layer number="45" name="Holes" color="7" fill="1" visible="no" active="yes"/>
+<layer number="45" name="Holes" color="7" fill="1" visible="yes" active="yes"/>
 <layer number="46" name="Milling" color="3" fill="1" visible="no" active="yes"/>
 <layer number="47" name="Measures" color="7" fill="1" visible="no" active="yes"/>
@@
 V1.0 Greg Tighe
 Lazer Tag</text>
+<hole x="85.09" y="62.23" drill="3.2"/>
+<hole x="3.81" y="62.23" drill="3.2"/>
 </plain>
 <attributes>
@@
 <wire x1="59.69" y1="7.62" x2="59.69" y2="15.11" width="0.4064" layer="1"/>
 <wire x1="60.96" y1="6.35" x2="59.69" y2="7.62" width="0.4064" layer="1"/>
-<wire x1="50.165" y1="60.96" x2="24.13" y2="60.96" width="0.4064" layer="1"/>
-<wire x1="50.8" y1="61.595" x2="50.165" y2="60.96" width="0.4064" layer="1"/>
-<wire x1="61.2775" y1="61.595" x2="50.8" y2="61.595" width="0.4064" layer="1"/>
+<wire x1="48.895" y1="60.96" x2="24.13" y2="60.96" width="0.4064" layer="1"/>
+<wire x1="49.53" y1="61.595" x2="48.895" y2="60.96" width="0.4064" layer="1"/>
+<wire x1="61.2775" y1="61.595" x2="49.53" y2="61.595" width="0.4064" layer="1"/>
 <wire x1="61.9125" y1="61.595" x2="61.2775" y2="61.595" width="0.4064" layer="16"/>
 <wire x1="64.135" y1="59.3725" x2="61.9125" y2="61.595" width="0.4064" layer="16"/>
